File: Gardening/Smart_Garden/Design/Smart Garden.sch (EAGLE design)
At the start: 68 parts, among them IC1 7809DT, IC2 LM1117-3.3, IC3 7805DT, J1 AUDIO_JACK_TRRSSMD_RA, J2 AUDIO_JACK_TRRSSMD_RA, J3 AUDIO_JACK_TRRSSMD_RA, J4 AUDIO_JACK_TRRSSMD_RA, T1 BC847, T2 BC847, T3 BC847, T4 BC847, U1 ESP-32S, U4 MB6S, X1 22-23-2021, X2 22-23-2021, X3 22-23-2021, X4 22-23-2021, X5 22-23-2021

Commit message: Updated Smart Garden Project docomentation
Parts:
- removed X1, X2, X3, X4, X5: 22-23-2021, con-molex:22-23-2021
- added X10, X6, X7, X8, X9: (no value), con-wago-500:W237-102
Connections:
- net 1R1: now also X7-2.KL; no longer X1-1.S
- net 2R1: now also X8-2.KL; no longer X2-1.S
- net 3R1: now also X9-2.KL; no longer X3-1.S
- net 4R1: now also X10-2.KL; no longer X4-1.S
- net AC1: now also X6-1.KL; no longer X5-2.S
- net AC2: now also X6-2.KL; no longer X5-1.S
- net N$1: now also X10-1.KL; no longer X4-2.S
- net N$2: now also X9-1.KL; no longer X3-2.S
- net N$4: now also X8-1.KL; no longer X2-2.S
- net N$5: now also X7-1.KL; no longer X1-2.S
Changed lines of the file:
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@@
 <part name="U$5" library="SpaceDIY_actuators" deviceset="RELAY" device="PTH"/>
 <part name="OK1" library="optocoupler" deviceset="SFH618?*" device="6" technology="-4"/>
-<part name="X1" library="con-molex" library_urn="urn:adsk.eagle:library:165" deviceset="22-23-2021" device="" package3d_urn="urn:adsk.eagle:package:8078633/1"/>
-<part name="X2" library="con-molex" library_urn="urn:adsk.eagle:library:165" deviceset="22-23-2021" device="" package3d_urn="urn:adsk.eagle:package:8078633/1"/>
-<part name="X3" library="con-molex" library_urn="urn:adsk.eagle:library:165" deviceset="22-23-2021" device="" package3d_urn="urn:adsk.eagle:package:8078633/1"/>
-<part name="X4" library="con-molex" library_urn="urn:adsk.eagle:library:165" deviceset="22-23-2021" device="" package3d_urn="urn:adsk.eagle:package:8078633/1"/>
 <part name="T1" library="transistor" library_urn="urn:adsk.eagle:library:402" deviceset="BC847" device="" package3d_urn="urn:adsk.eagle:package:28738/2"/>
 <part name="D2" library="diode" deviceset="DIODE-" device="SOD123"/>
@@
 <part name="H4" library="holes" deviceset="MOUNT-PAD-ROUND" device="3.0" value="MOUNT-PAD-ROUND3.0"/>
 <part name="GND20" library="SparkFun" deviceset="GND" device=""/>
-<part name="X5" library="con-molex" library_urn="urn:adsk.eagle:library:165" deviceset="22-23-2021" device="" package3d_urn="urn:adsk.eagle:package:8078633/1"/>
 <part name="J1" library="SparkFun-Connectors" deviceset="AUDIO_JACK_TRRS" device="SMD_RA"/>
 <part name="J2" library="SparkFun-Connectors" deviceset="AUDIO_JACK_TRRS" device="SMD_RA"/>
@@
 <part name="L4" library="SpaceDIY_passive_components" deviceset="LED1206" device="" value="Blue"/>
 <part name="L5" library="SpaceDIY_passive_components" deviceset="LED1206" device="" value="Blue"/>
+<part name="X6" library="con-wago-500" library_urn="urn:adsk.eagle:library:195" deviceset="W237-102" device="" package3d_urn="urn:adsk.eagle:package:10688/1"/>
+<part name="X7" library="con-wago-500" library_urn="urn:adsk.eagle:library:195" deviceset="W237-102" device="" package3d_urn="urn:adsk.eagle:package:10688/1"/>
+<part name="X8" library="con-wago-500" library_urn="urn:adsk.eagle:library:195" deviceset="W237-102" device="" package3d_urn="urn:adsk.eagle:package:10688/1"/>
+<part name="X9" library="con-wago-500" library_urn="urn:adsk.eagle:library:195" deviceset="W237-102" device="" package3d_urn="urn:adsk.eagle:package:10688/1"/>
+<part name="X10" library="con-wago-500" library_urn="urn:adsk.eagle:library:195" deviceset="W237-102" device="" package3d_urn="urn:adsk.eagle:package:10688/1"/>
 </parts>
 <sheets>
@@
 <attribute name="VALUE" x="46.355" y="88.9" size="1.778" layer="96"/>
 </instance>
-<instance part="X1" gate="-1" x="109.22" y="101.6" smashed="yes" rot="R180"/>
-<instance part="X1" gate="-2" x="111.76" y="91.44" smashed="yes"/>
-<instance part="X2" gate="-1" x="109.22" y="66.04" smashed="yes" rot="R180"/>
-<instance part="X2" gate="-2" x="111.76" y="55.88" smashed="yes"/>
-<instance part="X3" gate="-1" x="215.9" y="101.6" smashed="yes" rot="R180"/>
-<instance part="X3" gate="-2" x="218.44" y="91.44" smashed="yes"/>
-<instance part="X4" gate="-1" x="215.9" y="66.04" smashed="yes" rot="R180"/>
-<instance part="X4" gate="-2" x="218.44" y="55.88" smashed="yes"/>
 <instance part="T1" gate="G$1" x="81.28" y="83.82" smashed="yes">
 <attribute name="NAME" x="71.12" y="91.44" size="1.778" layer="95"/>
@@
 <attribute name="VALUE" x="248.92" y="27.94" size="1.778" layer="96"/>
 </instance>
-<instance part="X5" gate="-1" x="20.32" y="144.78" smashed="yes" rot="R180">
-<attribute name="NAME" x="17.78" y="145.542" size="1.524" layer="95" rot="R180"/>
-<attribute name="VALUE" x="21.082" y="143.383" size="1.778" layer="96" rot="R180"/>
-</instance>
-<instance part="X5" gate="-2" x="20.32" y="160.02" smashed="yes" rot="R180"/>
 <instance part="J1" gate="G$1" x="236.22" y="101.6" smashed="yes">
 <attribute name="NAME" x="231.14" y="107.188" size="1.778" layer="95" font="vector"/>
@@
 <attribute name="NAME" x="143.51" y="53.78" size="1.778" layer="95" align="center"/>
 <attribute name="VALUE" x="144.78" y="47.8" size="1.778" layer="96" align="center"/>
+</instance>
+<instance part="X6" gate="-1" x="17.78" y="160.02" smashed="yes">
+<attribute name="NAME" x="17.78" y="160.909" size="1.778" layer="95" rot="R180"/>
+</instance>
+<instance part="X6" gate="-2" x="17.78" y="144.78" smashed="yes">
+<attribute name="VALUE" x="15.24" y="141.097" size="1.778" layer="96"/>
+<attribute name="NAME" x="17.78" y="145.669" size="1.778" layer="95" rot="R180"/>
+</instance>
+<instance part="X7" gate="-1" x="114.3" y="91.44" smashed="yes" rot="R180">
+<attribute name="NAME" x="114.3" y="90.551" size="1.778" layer="95"/>
+</instance>
+<instance part="X7" gate="-2" x="106.68" y="101.6" smashed="yes">
+<attribute name="VALUE" x="104.14" y="97.917" size="1.778" layer="96"/>
+<attribute name="NAME" x="106.68" y="102.489" size="1.778" layer="95" rot="R180"/>
+</instance>
+<instance part="X8" gate="-1" x="114.3" y="55.88" smashed="yes" rot="R180">
+<attribute name="NAME" x="114.3" y="54.991" size="1.778" layer="95"/>
+</instance>
+<instance part="X8" gate="-2" x="106.68" y="66.04" smashed="yes">
+<attribute name="VALUE" x="104.14" y="62.357" size="1.778" layer="96"/>
+<attribute name="NAME" x="106.68" y="66.929" size="1.778" layer="95" rot="R180"/>
+</instance>
+<instance part="X9" gate="-1" x="220.98" y="91.44" smashed="yes" rot="R180">
+<attribute name="NAME" x="220.98" y="90.551" size="1.778" layer="95"/>
+</instance>
+<instance part="X9" gate="-2" x="213.36" y="101.6" smashed="yes">
+<attribute name="VALUE" x="210.82" y="97.917" size="1.778" layer="96"/>
+<attribute name="NAME" x="213.36" y="102.489" size="1.778" layer="95" rot="R180"/>
+</instance>
+<instance part="X10" gate="-1" x="220.98" y="55.88" smashed="yes" rot="R180">
+<attribute name="NAME" x="220.98" y="54.991" size="1.778" layer="95"/>
+</instance>
+<instance part="X10" gate="-2" x="213.36" y="66.04" smashed="yes">
+<attribute name="VALUE" x="210.82" y="62.357" size="1.778" layer="96"/>
+<attribute name="NAME" x="213.36" y="66.929" size="1.778" layer="95" rot="R180"/>
 </instance>
 </instances>
@@
 <wire x1="22.86" y1="160.02" x2="34.29" y2="160.02" width="0.1524" layer="91"/>
 <label x="22.86" y="161.29" size="1.778" layer="95"/>
-<pinref part="X5" gate="-2" pin="S"/>
+<pinref part="X6" gate="-1" pin="KL"/>
 </segment>
 </net>
@@
 <wire x1="34.29" y1="144.78" x2="22.86" y2="144.78" width="0.1524" layer="91"/>
 <label x="22.86" y="146.05" size="1.778" layer="95"/>
-<pinref part="X5" gate="-1" pin="S"/>
+<pinref part="X6" gate="-2" pin="KL"/>
 </segment>
 </net>
@@
 </segment>
 <segment>
-<pinref part="X1" gate="-1" pin="S"/>
 <wire x1="114.3" y1="101.6" x2="111.76" y2="101.6" width="0.1524" layer="91"/>
 <label x="111.76" y="101.6" size="1.778" layer="95"/>
+<pinref part="X7" gate="-2" pin="KL"/>
 </segment>
 </net>
@@
 <segment>
 <pinref part="U$5" gate="G$1" pin="SWOPEN"/>
-<pinref part="X4" gate="-2" pin="S"/>
 <wire x1="215.9" y1="55.88" x2="210.82" y2="55.88" width="0.1524" layer="91"/>
+<pinref part="X10" gate="-1" pin="KL"/>
 </segment>
 </net>
@@
 <segment>
 <pinref part="U$4" gate="G$1" pin="SWOPEN"/>
-<pinref part="X3" gate="-2" pin="S"/>
 <wire x1="215.9" y1="91.44" x2="210.82" y2="91.44" width="0.1524" layer="91"/>
+<pinref part="X9" gate="-1" pin="KL"/>
 </segment>
 </net>
@@
 <segment>
 <pinref part="U$3" gate="G$1" pin="SWOPEN"/>
-<pinref part="X2" gate="-2" pin="S"/>
 <wire x1="109.22" y1="55.88" x2="104.14" y2="55.88" width="0.1524" layer="91"/>
+<pinref part="X8" gate="-1" pin="KL"/>
 </segment>
 </net>
@@
 <segment>
 <pinref part="U$2" gate="G$1" pin="SWOPEN"/>
-<pinref part="X1" gate="-2" pin="S"/>
 <wire x1="109.22" y1="91.44" x2="104.14" y2="91.44" width="0.1524" layer="91"/>
+<pinref part="X7" gate="-1" pin="KL"/>
 </segment>
 </net>
@@
 </segment>
 <segment>
-<pinref part="X2" gate="-1" pin="S"/>
 <wire x1="114.3" y1="66.04" x2="111.76" y2="66.04" width="0.1524" layer="91"/>
 <label x="111.76" y="66.04" size="1.778" layer="95"/>
+<pinref part="X8" gate="-2" pin="KL"/>
 </segment>
 </net>
@@
 </segment>
 <segment>
-<pinref part="X3" gate="-1" pin="S"/>
 <wire x1="220.98" y1="101.6" x2="218.44" y2="101.6" width="0.1524" layer="91"/>
 <label x="218.44" y="101.6" size="1.778" layer="95"/>
+<pinref part="X9" gate="-2" pin="KL"/>
 </segment>
 </net>
@@
 </segment>
 <segment>
-<pinref part="X4" gate="-1" pin="S"/>
 <wire x1="218.44" y1="66.04" x2="220.98" y2="66.04" width="0.1524" layer="91"/>
 <label x="218.44" y="66.04" size="1.778" layer="95"/>
-</segment>
-</net>
+<pinref part="X10" gate="-2" pin="KL"/>
+</segment>
+</net>

Commit message: First commit to Smart Garden V1.1.0, changes apply mainly to schematics:  * Relay 5V supply  * Removed 220-24VAC transformator  * Staged power supply regulation with 12V step  * Push-buttons connection pins added
Parts:
- removed D1: (no value), diode:DIODE-SOD123
- removed U$1: TRANSFORMADOR_PE3010-M, SpaceDIY_special_components:TRANSFORMADOR_PE3010-M
- added C6, C7, C8: 100nF, SpaceDIY_passive_components:C1206
- added IC4: 7812DT, adafruit:7812DT
- added JP2, JP3, JP4, JP5: (no value), adafruit:PINHD-1X3
- added JP6: Power_switch, SpaceDIY_connectors:PINHD-1X4
- added SJ1: (no value), jumper:SJ2W
- added SJ2: (no value), SpaceDIY_connectors:SJ3W
- C1: device resistor:CPOL-USCT7343 -> rcl:CPOL-USD/7343-31R
Connections:
- removed net 24VDC: C1.+, D1.C, IC1.VI, IC3.VI, U4.+
- removed net AC1: U$1.P2, X6-1.KL
- removed net AC2: U$1.P1, X6-2.KL
- removed net N$10: D3.C, OK2.COL, U$3.COIL1
- removed net N$14: D4.C, OK3.COL, U$4.COIL1
- removed net N$18: D5.C, OK4.COL, U$5.COIL1
- new net 12V: C7.1, IC4.VO, S2.3, S3.3, S4.3, S5.3, SJ1.1, SJ2.4
- new net 24V: C1.+, C6.1, IC4.VI, SJ1.3, SJ2.3, U4.+
- new net IO3: JP3.3
- new net N$30: IC1.VI, SJ1.2
- new net N$32: IC3.VI, SJ2.1
- net 24V1: now also JP6.3; no longer U$1.S2
- net 24V2: now also X6-2.KL; no longer U$1.S1
- net 3V3: now also JP6.2; no longer S2.5, S3.5, S4.5, S5.5
- net 5V: now also D2.C, D3.C, D4.C, D5.C, OK1.COL, OK2.COL, OK3.COL, OK4.COL, S2.5, S3.5, S4.5, S5.5, U$2.COIL1, U$3.COIL1, U$4.COIL1, U$5.COIL1; no longer D1.A, S2.4, S3.4, S4.4, S5.4
- net 9V: now also C8.1, S2.4, S3.4, S4.4, S5.4, SJ2.2; no longer S2.3, S3.3, S4.3, S5.3
- net GND: now also C6.2, C7.2, C8.2, IC4.GND, JP2.1, JP3.1, JP4.1, JP5.1, JP6.1
- net IO12: now also JP2.2
- net IO13: now also JP3.2
- net IO15: now also JP5.3
- net IO2: now also JP2.3
- net IO23: now also JP4.2
- net IO25: now also JP5.2
- net IO5: now also JP4.3
- net N$1: now also U$3.SWCLOSE, X8-1.KL; no longer U$5.SWOPEN, X10-1.KL
- net N$2: now also U$2.SWCLOSE, X7-1.KL; no longer U$4.SWOPEN, X9-1.KL
- net N$4: now also U$4.SWCLOSE, X9-1.KL; no longer U$3.SWOPEN, X8-1.KL
- net N$5: now also U$5.SWCLOSE, X10-1.KL; no longer U$2.SWOPEN, X7-1.KL
- net N$6: now also JP6.4, X6-1.KL; no longer D2.C, OK1.COL, U$2.COIL1
Other:
- note added: "Flash"
- note added: "PB_In_1"
- note added: "PB_In_2"
- note added: "PB_In_3"
- note added: "PB_In_4"
- note added: "PB_LED_1"
- note added: "PB_LED_2"
- note added: "PB_LED_3"
- note added: "PB_LED_4"
- note added: "RST"
- note added: "SCL"
- note added: "SDA"
- moved on the sheet: C1, C2, C3, C4, C5, IC1, IC2, IC3, L1, R1, R11, R2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

Commit message: Updated Design files
Connections:
- removed net IO3: JP3.3
- net 1R1: now also X7-1.KL; no longer X7-2.KL
- net 2R1: now also X8-1.KL; no longer X8-2.KL
- net IO13: no longer J3.RING2
- net IO14: now also J3.RING2
- net N$1: now also X8-2.KL; no longer X8-1.KL
- net N$2: now also X7-2.KL; no longer X7-1.KL
- net RX: now also JP3.3
Other:
- note added: "By J.G.Aguado"
- note added: "V1.1"
- moved on the sheet: X7-1, X7-2, X8-1, X8-2
Changed lines of the file:
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@@
 <text x="162.56" y="124.46" size="1.778" layer="91">PB_LED_2</text>
 <text x="170.18" y="160.02" size="1.778" layer="91">RST</text>
+<text x="248.92" y="5.08" size="2.1844" layer="94">V1.1</text>
+<text x="218.44" y="15.24" size="2.1844" layer="94">By J.G.Aguado</text>
 </plain>
 <instances>
 <instance part="FRAME1" gate="G$1" x="0" y="0" smashed="yes">
-<attribute name="DRAWING_NAME" x="217.17" y="15.24" size="2.54" layer="94" font="vector"/>
+<attribute name="DRAWING_NAME" x="217.17" y="20.32" size="2.54" layer="94" font="vector"/>
 <attribute name="LAST_DATE_TIME" x="217.17" y="10.16" size="2.286" layer="94" font="vector"/>
 <attribute name="SHEET" x="230.505" y="5.08" size="2.54" layer="94" font="vector"/>
@@
 <attribute name="NAME" x="12.7" y="148.209" size="1.778" layer="95" rot="R180"/>
 </instance>
-<instance part="X7" gate="-1" x="111.76" y="101.6" smashed="yes" rot="R180">
+<instance part="X7" gate="-1" x="106.68" y="91.44" smashed="yes">
+<attribute name="NAME" x="106.68" y="92.329" size="1.778" layer="95" rot="R180"/>
+</instance>
+<instance part="X7" gate="-2" x="111.76" y="101.6" smashed="yes" rot="R180">
+<attribute name="VALUE" x="114.3" y="105.283" size="1.778" layer="96" rot="R180"/>
 <attribute name="NAME" x="111.76" y="100.711" size="1.778" layer="95"/>
 </instance>
-<instance part="X7" gate="-2" x="106.68" y="91.44" smashed="yes">
-<attribute name="VALUE" x="104.14" y="87.757" size="1.778" layer="96"/>
-<attribute name="NAME" x="106.68" y="92.329" size="1.778" layer="95" rot="R180"/>
-</instance>
-<instance part="X8" gate="-1" x="111.76" y="66.04" smashed="yes" rot="R180">
+<instance part="X8" gate="-1" x="106.68" y="55.88" smashed="yes">
+<attribute name="NAME" x="106.68" y="56.769" size="1.778" layer="95" rot="R180"/>
+</instance>
+<instance part="X8" gate="-2" x="111.76" y="66.04" smashed="yes" rot="R180">
+<attribute name="VALUE" x="114.3" y="69.723" size="1.778" layer="96" rot="R180"/>
 <attribute name="NAME" x="111.76" y="65.151" size="1.778" layer="95"/>
-</instance>
-<instance part="X8" gate="-2" x="106.68" y="55.88" smashed="yes">
-<attribute name="VALUE" x="104.14" y="52.197" size="1.778" layer="96"/>
-<attribute name="NAME" x="106.68" y="56.769" size="1.778" layer="95" rot="R180"/>
 </instance>
 <instance part="X9" gate="-1" x="218.44" y="101.6" smashed="yes" rot="R180">
@@
 </segment>
 <segment>
-<wire x1="114.3" y1="91.44" x2="111.76" y2="91.44" width="0.1524" layer="91"/>
+<pinref part="X7" gate="-1" pin="KL"/>
+<wire x1="111.76" y1="91.44" x2="114.3" y2="91.44" width="0.1524" layer="91"/>
 <label x="111.76" y="91.44" size="1.778" layer="95"/>
-<pinref part="X7" gate="-2" pin="KL"/>
 </segment>
 </net>
@@
 </segment>
 <segment>
-<wire x1="114.3" y1="55.88" x2="111.76" y2="55.88" width="0.1524" layer="91"/>
+<pinref part="X8" gate="-1" pin="KL"/>
+<wire x1="111.76" y1="55.88" x2="114.3" y2="55.88" width="0.1524" layer="91"/>
 <label x="111.76" y="55.88" size="1.778" layer="95"/>
-<pinref part="X8" gate="-2" pin="KL"/>
 </segment>
 </net>
@@
 <label x="177.8" y="134.62" size="1.778" layer="95"/>
 </segment>
+<segment>
+<pinref part="J3" gate="G$1" pin="RING2"/>
+<wire x1="248.92" y1="66.04" x2="241.3" y2="66.04" width="0.1524" layer="91"/>
+<label x="243.84" y="66.04" size="1.778" layer="95"/>
+</segment>
 </net>
 <net name="IO12" class="0">
@@
 <wire x1="177.8" y1="124.46" x2="187.96" y2="124.46" width="0.1524" layer="91"/>
 <label x="177.8" y="124.46" size="1.778" layer="95"/>
-</segment>
-<segment>
-<pinref part="J3" gate="G$1" pin="RING2"/>
-<wire x1="248.92" y1="66.04" x2="241.3" y2="66.04" width="0.1524" layer="91"/>
-<label x="243.84" y="66.04" size="1.778" layer="95"/>
 </segment>
 <segment>
@@
 <wire x1="30.48" y1="111.76" x2="20.32" y2="111.76" width="0.1524" layer="91"/>
 <label x="25.4" y="111.76" size="1.778" layer="95"/>
+</segment>
+<segment>
+<pinref part="JP3" gate="A" pin="3"/>
+<wire x1="170.18" y1="33.02" x2="180.34" y2="33.02" width="0.1524" layer="91"/>
+<label x="175.26" y="33.02" size="1.778" layer="95"/>
 </segment>
 </net>
@@
 </segment>
 </net>
-<net name="IO3" class="0">
-<segment>
-<pinref part="JP3" gate="A" pin="3"/>
-<wire x1="170.18" y1="33.02" x2="180.34" y2="33.02" width="0.1524" layer="91"/>
-<label x="175.26" y="33.02" size="1.778" layer="95"/>
-</segment>
-</net>
-<net name="N$1" class="0">
-<segment>
-<pinref part="U$3" gate="G$1" pin="SWCLOSE"/>
-<pinref part="X8" gate="-1" pin="KL"/>
-<wire x1="106.68" y1="66.04" x2="104.14" y2="66.04" width="0.1524" layer="91"/>
-</segment>
-</net>
-<net name="N$2" class="0">
-<segment>
-<pinref part="U$2" gate="G$1" pin="SWCLOSE"/>
-<pinref part="X7" gate="-1" pin="KL"/>
-<wire x1="106.68" y1="101.6" x2="104.14" y2="101.6" width="0.1524" layer="91"/>
-</segment>
-</net>
 <net name="N$4" class="0">
 <segment>
@@
 </segment>
 </net>
+<net name="N$2" class="0">
+<segment>
+<pinref part="U$2" gate="G$1" pin="SWCLOSE"/>
+<pinref part="X7" gate="-2" pin="KL"/>
+<wire x1="106.68" y1="101.6" x2="104.14" y2="101.6" width="0.1524" layer="91"/>
+</segment>
+</net>
+<net name="N$1" class="0">
+<segment>
+<pinref part="U$3" gate="G$1" pin="SWCLOSE"/>
+<pinref part="X8" gate="-2" pin="KL"/>
+<wire x1="106.68" y1="66.04" x2="104.14" y2="66.04" width="0.1524" layer="91"/>
+</segment>
+</net>
