File: Gardening/WMF_Ambient_SmartPot/Design/WMF Ambient SmartPot_B.brd (EAGLE design)
At the start: 30 x 56.5 mm, 45 parts, among them IC1 LM1117-5.0, IC2 LM1117-3.3, U1 ESP-32S

Commit message: Updated Design files WMF Ambient SmartPot_B
Parts:
- removed JP5: Pot1, SpaceDIY_connectors:1X04
- removed JP6: Pot2, SpaceDIY_connectors:1X04
- removed JP8: Water Tank, SpaceDIY_connectors:1X03
- added JP2: Serial, SpaceDIY_connectors:1X04
- added R3: 10k, SpaceDIY_passive_components:1206
- added S1: MOMENTARY-SWITCH-SPST-SMD-6.0X3.5MM, SparkFun-Switches:TACTILE_SWITCH_SMD_6.0X3.5MM
- CN1: device SpaceDIY_connectors:DCJACK_2MM_PTH -> SpaceDIY_connectors:DCJACK_2MM_PTH-2
- moved R8 0.15 mm to (28.0, 71.9)
Connections:
- net 12V: now also JP2.3; no longer IC2.3
- net 3V3: now also JP2.1, R3.1; no longer JP5.4, JP6.4
- net 5V: now also IC2.3, JP2.2
- net EN: now also R3.2, S1.2
- net GND: now also JP2.4, S1.1; no longer JP5.3, JP6.3, JP8.2
- net IO12: no longer JP6.2
- net IO13: no longer JP6.1
- net IO14: no longer JP8.1
- net IO15: no longer JP5.1
- net IO2: no longer JP5.2
- net IO27: no longer JP8.3
Routing:
- net IO27: track 76.5 -> 51.6 mm, vias 4 -> 3
- net IO14: track 76.5 -> 53.9 mm
- net 5V: track 83.3 -> 97.6 mm, vias 3 -> 4
- net EN: track 0.00 -> 13.3 mm, vias 0 -> 1
- net 3V3: track 122.4 -> 109.8 mm, vias 8 -> 5
- net IO13: track 76.9 -> 64.5 mm
- net IO12: track 63.2 -> 52.1 mm, vias 2 -> 1
- net GND: track 15.9 -> 22.2 mm, vias 17 -> 21
- net 12V: track 56.0 -> 51.0 mm
- net IO2: track 45.2 -> 42.0 mm
- net IO21: track 35.9 -> 34.0 mm
- net IO22: track 44.4 -> 44.0 mm, vias 4 -> 2
- net IO15: track 52.8 -> 52.9 mm, vias 1 -> 2
Other:
- outline, holes or cut-outs redrawn
- board text added: "+"
- board text added: "-"
- board text added: "12"
- board text added: "3"
- board text added: "5"
- board text added: "V1.1"
