File: Gardening/WMF_Ambient_SmartPot/Design/WMF Ambient SmartPot_B.sch (EAGLE design)
At the start: 68 parts, among them IC1 LM1117-5.0, IC2 LM1117-3.3, J1 AUDIO_JACK_TRRSSMD_RA, J2 AUDIO_JACK_TRRSSMD_RA, U1 ESP-32S

Commit message: Changed the panelized design to individual boards design
Parts:
- removed H1, H2: MOUNT-PAD-ROUND2.8, holes:MOUNT-PAD-ROUND2.8
- removed J1, J2: AUDIO_JACK_TRRSSMD_RA, SparkFun-Connectors:AUDIO_JACK_TRRSSMD_RA
- removed JP7: BME280, SpaceDIY_connectors:PINHD-1X4
- removed R3: 10k, SpaceDIY_passive_components:R1206
- removed SJ1, SJ2: (no value), jumper:SJ2W
- removed TP1, TP12, TP16, TP17, TP20, TP21, TP23, TP6, TP7, TP8, TP9: TPTP15SQ, testpad:TPTP15SQ
- removed U$2, U$3, U$4, U$5: OVAL_3MM_HOLE, SpaceDIY_connectors:OVAL_3MM_HOLE
Connections:
- removed net 3V3_W: SJ2.2, U$4.P$1
- removed net IN_B: SJ2.3
- removed net IN_T: SJ2.1
- removed net OUT_B: SJ1.3
- removed net OUT_T: SJ1.1
- removed net OUT_W: SJ1.2, U$5.P$1
- removed net S12: J1.TIP, TP16.TP
- removed net S13: J1.RING2, TP17.TP
- removed net S14: TP12.TP, U$2.P$1
- removed net S15: J2.RING2, TP21.TP
- removed net S2: J2.TIP, TP20.TP
- removed net S27: R3.1, TP23.TP, U$3.P$1
- removed net S3V3: J1.RING1, J2.RING1, JP7.4, TP6.TP
- removed net SSCL: JP7.2, TP8.TP
- removed net SSDA: JP7.1, TP9.TP
- removed net TOUCH: H1.MOUNT, H2.MOUNT, TP1.TP
- net GND: no longer J1.EARTH, J2.EARTH, JP7.3, R3.2, TP7.TP
Other:
- moved on the sheet: C1, C2, C3, C4, C5, CN1, IC1, IC2, JP1, JP10, JP11, JP4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

Commit message: Updated Design files WMF Ambient SmartPot_B
Parts:
- removed JP5: Pot1, SpaceDIY_connectors:PINHD-1X4
- removed JP6: Pot2, SpaceDIY_connectors:PINHD-1X4
- removed JP8: Water Tank, SpaceDIY_connectors:PINHD-1X3
- added JP2: Serial, SpaceDIY_connectors:PINHD-1X4
- added R3: 10k, SpaceDIY_passive_components:R1206
- added S1: MOMENTARY-SWITCH-SPST-SMD-6.0X3.5MM, SparkFun-Switches:MOMENTARY-SWITCH-SPST-SMD-6.0X3.5MM
- CN1: device SpaceDIY_connectors:DCBARRELPTH -> SpaceDIY_connectors:DCBARREL-2
Connections:
- net 12V: now also JP2.3; no longer IC2.IN
- net 3V3: now also JP2.1, R3.1; no longer JP5.4, JP6.4
- net 5V: now also IC2.IN, JP2.2
- net EN: now also R3.2, S1.2
- net GND: now also JP2.4, S1.1; no longer JP5.3, JP6.3, JP8.2
- net IO12: no longer JP6.2
- net IO13: no longer JP6.1
- net IO14: no longer JP8.1
- net IO15: no longer JP5.1
- net IO2: no longer JP5.2
- net IO27: no longer JP8.3
Other:
- moved on the sheet: C3, C5, IC2, L1, R1
